File: EAGLE/projects/input switch/input_switch2_bad.brd (EAGLE design)
At the start: 50 x 100 mm, 55 parts, among them U1 NE5532P, U2 NE5532P

Commit message: input
Parts:
- removed R_GND1, R_GND2, R_PS1, R_PS2: 100, rcl:0207/7
- added C7_1, C7_2: 220u, rcl:E5-10,5
- added U3: NE5532P, ne5532:DIP254P762X508-8
- U1, U2: value NE5532P -> NE5532AD8G; device ne5532:DIP254P762X508-8 -> ne5532:SOIC127P600X175-8N
- moved C6_2 117.1 mm to (41.9, 38.1), turned to 90 degrees
- moved C3_2_BP 116.1 mm to (39.4, 72.4), turned to 270 degrees
- moved R2_2 109.7 mm to (40.6, 87.6), turned to 90 degrees
- moved L_2 107.4 mm to (30.5, 95.2)
- moved R5_2 101.7 mm to (33.0, 64.8), turned to 270 degrees
- moved R4_2 94.4 mm to (44.5, 86.4), turned to 270 degrees
- moved C6_1 93.4 mm to (27.9, 38.1), turned to 90 degrees
- moved C5_2 91.2 mm to (35.6, 36.8), turned to 90 degrees
- moved U2 89.3 mm to (40.6, 50.8)
- moved A_OUT_2 88.9 mm to (35.6, 5.08)
- moved C4_2 87.0 mm to (44.5, 78.7)
- moved L_1 81.7 mm to (7.62, 95.2)
- moved C3_1_BP 80.7 mm to (16.5, 72.4), turned to 270 degrees
- moved R1_2 79.1 mm to (29.2, 87.6), turned to 90 degrees
- moved R2_1 77.9 mm to (17.8, 87.6), turned to 90 degrees
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Connections:
- removed net AGND: A_OUT_1.2, A_OUT_2.2, C1_2.2, C4_1.2, C4_2.2, R3_2.1, R4_1.1, R4_2.1, R5_1.1, R5_2.1, R6_1.1, R6_2.1, R_GND1.1, R_GND2.1
- removed net N$17: -15V.1, R_PS2.2
- removed net N$25: +15V.1, R_PS1.2
- removed net N$41: C1_1.2, R3_1.1
- new net VCC+: U3.8
- new net VCC-: U3.4
- net +15V: now also +15V.1; no longer R_PS1.1
- net -15V: now also -15V.1; no longer R_PS2.1
- net GND: now also A_OUT_1.2, A_OUT_2.2, C1_1.2, C1_2.2, C4_1.2, C4_2.2, R3_1.1, R3_2.1, R4_1.1, R4_2.1, R5_1.1, R5_2.1, R6_1.1, R6_2.1; no longer R_GND1.2, R_GND2.2
- net N$18: now also C7_1.-
- net N$37: now also C7_1.+, C7_2.+
- net N$38: now also C7_2.-
Routing:
- net GND: track 0.00 -> 117.2 mm
- net N$3: track 0.00 -> 18.6 mm
- net N$24: track 0.00 -> 18.6 mm
- net N$23: track 0.00 -> 18.6 mm
- net N$6: track 0.00 -> 18.6 mm
- net N$27: track 0.00 -> 14.5 mm
- net N$26: track 0.00 -> 14.5 mm
- net N$4: track 0.00 -> 14.5 mm
- net N$20: track 0.00 -> 14.5 mm
- net N$21: track 0.00 -> 3.81 mm
- net N$2: track 0.00 -> 3.81 mm
- net N$1: track 0.00 -> 3.81 mm
