File: EAGLE/projects/input switch/input_switch2.sch (EAGLE design)
At the start: 57 parts, among them U1 NE5532P, U2 NE5532P

Commit message: Input Board done
Parts:
- added C1, C2: (no value), rcl:C-USC1206
- added J1: J12MM, jumper:J12MM
- added J2: J25MM, jumper:J25MM
- added SJ1, SJ2, SJ3, SJ4: (no value), jumper:SJ
Connections:
- new net N$44: J2.2, RELAY2.10
- net +15V: now also C1.1
- net -15V: now also C2.2
- net AGND: now also C1_1.2, R3_1.1, R8_1.1, R8_2.1, R9_1.1, R9_2.1, SJ1.1, SJ1.2, SJ2.1, SJ2.2, SJ3.1, SJ3.2, SJ4.1, SJ4.2
- net GND: now also C1.2, C2.1; no longer R8_1.1, R8_2.1, R9_1.1, R9_2.1
- net N$37: now also J1.2; no longer RELAY2.1
- net N$38: now also J2.1; no longer RELAY2.10
- net N$41: now also J1.1, RELAY2.1; no longer C1_1.2, R3_1.1
Other:
- moved on the sheet: +15V, D2, Q1, Q2, R7_1, R7_2, RGND3, RGND4, RLY_CTRL, R_PS1

Commit message: a lot
Parts:
- removed SJ1, SJ2, SJ3, SJ4: (no value), jumper:SJ
- added R1: 100, rcl:R-US_R1206
Connections:
- net AGND: now also R1.1; no longer SJ1.1, SJ1.2, SJ2.1, SJ2.2, SJ3.1, SJ3.2, SJ4.1, SJ4.2
- net GND: now also R1.2
Changed lines of the file:
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@@
 <part name="J1" library="jumper" deviceset="J" device="12MM" value="J12MM"/>
 <part name="J2" library="jumper" deviceset="J" device="25MM" value="J25MM"/>
-<part name="SJ1" library="jumper" deviceset="SJ" device=""/>
-<part name="SJ2" library="jumper" deviceset="SJ" device=""/>
-<part name="SJ3" library="jumper" deviceset="SJ" device=""/>
-<part name="SJ4" library="jumper" deviceset="SJ" device=""/>
-<part name="AGND14" library="supply1" deviceset="AGND" device=""/>
-<part name="AGND15" library="supply1" deviceset="AGND" device=""/>
+<part name="R1" library="rcl" deviceset="R-US_" device="R1206" value="100"/>
+<part name="GND1" library="supply1" deviceset="GND" device=""/>
 </parts>
 <sheets>
@@
 <instance part="J1" gate="1" x="86.36" y="43.18" rot="R90"/>
 <instance part="J2" gate="1" x="106.68" y="43.18" rot="R270"/>
-<instance part="SJ1" gate="1" x="30.48" y="96.52"/>
-<instance part="SJ2" gate="1" x="30.48" y="88.9"/>
-<instance part="SJ3" gate="1" x="116.84" y="96.52"/>
-<instance part="SJ4" gate="1" x="116.84" y="88.9"/>
-<instance part="AGND14" gate="VR1" x="38.1" y="83.82"/>
-<instance part="AGND15" gate="VR1" x="109.22" y="83.82"/>
+<instance part="R1" gate="G$1" x="33.02" y="96.52"/>
+<instance part="GND1" gate="1" x="40.64" y="91.44"/>
 </instances>
 <busses>
@@
 <wire x1="-78.74" y1="10.16" x2="-78.74" y2="30.48" width="0.1524" layer="91"/>
 <wire x1="-78.74" y1="30.48" x2="-63.5" y2="30.48" width="0.1524" layer="91"/>
+</segment>
+<segment>
+<pinref part="R1" gate="G$1" pin="2"/>
+<pinref part="GND1" gate="1" pin="GND"/>
+<wire x1="38.1" y1="96.52" x2="40.64" y2="96.52" width="0.1524" layer="91"/>
+<wire x1="40.64" y1="96.52" x2="40.64" y2="93.98" width="0.1524" layer="91"/>
 </segment>
 </net>
@@
 <pinref part="RGND1" gate="G$1" pin="1"/>
 <pinref part="RGND2" gate="G$1" pin="1"/>
-<pinref part="SJ1" gate="1" pin="1"/>
+<pinref part="R1" gate="G$1" pin="1"/>
+<wire x1="25.4" y1="96.52" x2="27.94" y2="96.52" width="0.1524" layer="91"/>
 <junction x="25.4" y="96.52"/>
-<pinref part="SJ2" gate="1" pin="1"/>
 </segment>
 <segment>
@@
 <pinref part="RGND3" gate="G$1" pin="1"/>
 <pinref part="RGND4" gate="G$1" pin="1"/>
-<pinref part="SJ3" gate="1" pin="2"/>
-<junction x="121.92" y="96.52"/>
-<pinref part="SJ4" gate="1" pin="2"/>
 </segment>
 <segment>
@@
 <pinref part="AGND13" gate="VR1" pin="AGND"/>
 </segment>
-<segment>
-<pinref part="SJ1" gate="1" pin="2"/>
-<pinref part="AGND14" gate="VR1" pin="AGND"/>
-<wire x1="35.56" y1="96.52" x2="38.1" y2="96.52" width="0.1524" layer="91"/>
-<wire x1="38.1" y1="96.52" x2="38.1" y2="88.9" width="0.1524" layer="91"/>
-<pinref part="SJ2" gate="1" pin="2"/>
-<wire x1="38.1" y1="88.9" x2="38.1" y2="86.36" width="0.1524" layer="91"/>
-<wire x1="35.56" y1="88.9" x2="38.1" y2="88.9" width="0.1524" layer="91"/>
-<junction x="38.1" y="88.9"/>
-</segment>
-<segment>
-<pinref part="SJ3" gate="1" pin="1"/>
-<pinref part="AGND15" gate="VR1" pin="AGND"/>
-<wire x1="111.76" y1="96.52" x2="109.22" y2="96.52" width="0.1524" layer="91"/>
-<wire x1="109.22" y1="96.52" x2="109.22" y2="88.9" width="0.1524" layer="91"/>
-<pinref part="SJ4" gate="1" pin="1"/>
-<wire x1="109.22" y1="88.9" x2="109.22" y2="86.36" width="0.1524" layer="91"/>
-<wire x1="111.76" y1="88.9" x2="109.22" y2="88.9" width="0.1524" layer="91"/>
-<junction x="109.22" y="88.9"/>
-</segment>
-</net>
+</net>

Commit message: stuff
Parts:
- R8_1, R8_2, R9_1, R9_2: value 220k -> 330k
- renumbered A_OUT_1 to OUT1, A_OUT_2 to OUT2, L_1 to LEFT1, L_2 to LEFT2, R_1 to RIGHT1, R_2 to RIGHT2
