File: EAGLE/projects/EMI AC filter/EMI_filter.brd (EAGLE design)
At the start: 135.9 x 47.9 mm, 9 parts

Commit message: a lot
Routing:
- removed copper zone on layer 16, net GND
Other:
- board text removed: "GND"
- board text removed: "V+"
- board text removed: "V-"
Changed lines of the file:
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@@
 <layer number="14" name="Route14" color="1" fill="6" visible="no" active="no"/>
 <layer number="15" name="Route15" color="4" fill="6" visible="no" active="no"/>
-<layer number="16" name="Bottom" color="1" fill="1" visible="yes" active="yes"/>
-<layer number="17" name="Pads" color="2" fill="1" visible="yes" active="yes"/>
-<layer number="18" name="Vias" color="2" fill="1" visible="yes" active="yes"/>
-<layer number="19" name="Unrouted" color="6" fill="1" visible="yes" active="yes"/>
-<layer number="20" name="Dimension" color="15" fill="1" visible="yes" active="yes"/>
-<layer number="21" name="tPlace" color="7" fill="1" visible="yes" active="yes"/>
-<layer number="22" name="bPlace" color="7" fill="1" visible="yes" active="yes"/>
-<layer number="23" name="tOrigins" color="15" fill="1" visible="yes" active="yes"/>
-<layer number="24" name="bOrigins" color="15" fill="1" visible="yes" active="yes"/>
-<layer number="25" name="tNames" color="7" fill="1" visible="yes" active="yes"/>
-<layer number="26" name="bNames" color="7" fill="1" visible="yes" active="yes"/>
-<layer number="27" name="tValues" color="7" fill="1" visible="yes" active="yes"/>
-<layer number="28" name="bValues" color="7" fill="1" visible="yes" active="yes"/>
+<layer number="16" name="Bottom" color="1" fill="1" visible="no" active="yes"/>
+<layer number="17" name="Pads" color="2" fill="1" visible="no" active="yes"/>
+<layer number="18" name="Vias" color="2" fill="1" visible="no" active="yes"/>
+<layer number="19" name="Unrouted" color="6" fill="1" visible="no" active="yes"/>
+<layer number="20" name="Dimension" color="15" fill="1" visible="no" active="yes"/>
+<layer number="21" name="tPlace" color="7" fill="1" visible="no" active="yes"/>
+<layer number="22" name="bPlace" color="7" fill="1" visible="no" active="yes"/>
+<layer number="23" name="tOrigins" color="15" fill="1" visible="no" active="yes"/>
+<layer number="24" name="bOrigins" color="15" fill="1" visible="no" active="yes"/>
+<layer number="25" name="tNames" color="7" fill="1" visible="no" active="yes"/>
+<layer number="26" name="bNames" color="7" fill="1" visible="no" active="yes"/>
+<layer number="27" name="tValues" color="7" fill="1" visible="no" active="yes"/>
+<layer number="28" name="bValues" color="7" fill="1" visible="no" active="yes"/>
 <layer number="29" name="tStop" color="7" fill="3" visible="no" active="yes"/>
 <layer number="30" name="bStop" color="7" fill="6" visible="no" active="yes"/>
@@
 <layer number="37" name="tTest" color="7" fill="1" visible="no" active="yes"/>
 <layer number="38" name="bTest" color="7" fill="1" visible="no" active="yes"/>
-<layer number="39" name="tKeepout" color="4" fill="11" visible="yes" active="yes"/>
-<layer number="40" name="bKeepout" color="1" fill="11" visible="yes" active="yes"/>
-<layer number="41" name="tRestrict" color="4" fill="10" visible="yes" active="yes"/>
-<layer number="42" name="bRestrict" color="1" fill="10" visible="yes" active="yes"/>
-<layer number="43" name="vRestrict" color="2" fill="10" visible="yes" active="yes"/>
+<layer number="39" name="tKeepout" color="4" fill="11" visible="no" active="yes"/>
+<layer number="40" name="bKeepout" color="1" fill="11" visible="no" active="yes"/>
+<layer number="41" name="tRestrict" color="4" fill="10" visible="no" active="yes"/>
+<layer number="42" name="bRestrict" color="1" fill="10" visible="no" active="yes"/>
+<layer number="43" name="vRestrict" color="2" fill="10" visible="no" active="yes"/>
 <layer number="44" name="Drills" color="7" fill="1" visible="no" active="yes"/>
 <layer number="45" name="Holes" color="7" fill="1" visible="no" active="yes"/>
 <layer number="46" name="Milling" color="3" fill="1" visible="no" active="yes"/>
 <layer number="47" name="Measures" color="7" fill="1" visible="no" active="yes"/>
-<layer number="48" name="Document" color="7" fill="1" visible="yes" active="yes"/>
-<layer number="49" name="Reference" color="7" fill="1" visible="yes" active="yes"/>
-<layer number="51" name="tDocu" color="7" fill="1" visible="yes" active="yes"/>
-<layer number="52" name="bDocu" color="7" fill="1" visible="yes" active="yes"/>
+<layer number="48" name="Document" color="7" fill="1" visible="no" active="yes"/>
+<layer number="49" name="Reference" color="7" fill="1" visible="no" active="yes"/>
+<layer number="51" name="tDocu" color="7" fill="1" visible="no" active="yes"/>
+<layer number="52" name="bDocu" color="7" fill="1" visible="no" active="yes"/>
 <layer number="91" name="Nets" color="2" fill="1" visible="no" active="no"/>
 <layer number="92" name="Busses" color="1" fill="1" visible="no" active="no"/>
@@
 <wire x1="128.25" y1="45.39" x2="-7.62" y2="45.39" width="0" layer="20"/>
 <wire x1="-7.62" y1="45.39" x2="-7.62" y2="-2.54" width="0" layer="20"/>
-<dimension x1="37.465" y1="-6.35" x2="59.69" y2="-6.35" x3="48.5775" y3="48.26" textsize="1.778" layer="49"/>
 <rectangle x1="-5.08" y1="7.62" x2="7.62" y2="35.56" layer="49"/>
 <rectangle x1="113.03" y1="7.62" x2="125.73" y2="35.56" layer="49"/>
-<dimension x1="15.875" y1="30.48" x2="15.875" y2="12.065" x3="132.08" y3="21.2725" textsize="1.778" layer="49"/>
 <rectangle x1="27.305" y1="6.985" x2="69.215" y2="36.195" layer="49"/>
 <text x="51.435" y="0" size="1.778" layer="1" rot="R90">Matt Hengeveld
@@
 <text x="51.435" y="29.845" size="1.778" layer="1" rot="R90">AC EMI
   Filter</text>
-<text x="-3.81" y="24.13" size="1.778" layer="16" rot="MR270">GND</text>
-<text x="-2.54" y="41.275" size="1.778" layer="16" rot="MR0">V+</text>
-<text x="-2.54" y="-0.635" size="1.778" layer="16" rot="MR0">V-</text>
 </plain>
 <attributes>
@@
 <vertex x="58.42" y="44.45"/>
 <vertex x="54.61" y="40.64"/>
-<vertex x="54.61" y="26.67"/>
-<vertex x="57.15" y="24.13"/>
-<vertex x="93.98" y="24.13"/>
-<vertex x="100.33" y="30.48"/>
+<vertex x="54.61" y="30.48"/>
+<vertex x="57.15" y="27.94"/>
+<vertex x="96.52" y="27.94"/>
+<vertex x="99.06" y="30.48"/>
 <vertex x="110.49" y="30.48"/>
-<vertex x="114.3" y="26.67"/>
-<vertex x="123.19" y="26.67"/>
+<vertex x="113.03" y="27.94"/>
+<vertex x="124.46" y="27.94"/>
 <vertex x="127" y="30.48"/>
 </polygon>
@@
 <via x="119.38" y="13.335" extent="1-16" drill="1.5" diameter="2.54"/>
 <polygon width="0.4064" layer="1" spacing="0.4064" isolate="1.6764" thermals="no">
-<vertex x="123.19" y="16.51"/>
+<vertex x="124.46" y="15.24"/>
 <vertex x="127" y="12.7"/>
 <vertex x="127" y="2.54"/>
@@
 <vertex x="58.42" y="-1.27"/>
 <vertex x="54.61" y="2.54"/>
-<vertex x="54.61" y="16.51"/>
-<vertex x="57.15" y="19.05"/>
-<vertex x="93.98" y="19.05"/>
-<vertex x="100.33" y="12.7"/>
+<vertex x="54.61" y="12.7"/>
+<vertex x="57.15" y="15.24"/>
+<vertex x="96.52" y="15.24"/>
+<vertex x="99.06" y="12.7"/>
 <vertex x="110.49" y="12.7"/>
-<vertex x="114.3" y="16.51"/>
+<vertex x="113.03" y="15.24"/>
 </polygon>
 </signal>
@@
 <vertex x="-6.35" y="12.7"/>
 <vertex x="-3.81" y="15.24"/>
-<vertex x="12.7" y="15.24"/>
-<vertex x="16.51" y="19.05"/>
-<vertex x="39.37" y="19.05"/>
-<vertex x="43.18" y="15.24"/>
+<vertex x="39.37" y="15.24"/>
+<vertex x="43.18" y="11.43"/>
 <vertex x="43.18" y="2.54"/>
 <vertex x="39.37" y="-1.27"/>
@@
 <vertex x="-6.35" y="30.48"/>
 <vertex x="-3.81" y="27.94"/>
-<vertex x="12.7" y="27.94"/>
-<vertex x="16.51" y="24.13"/>
-<vertex x="39.37" y="24.13"/>
-<vertex x="43.18" y="27.94"/>
+<vertex x="39.37" y="27.94"/>
+<vertex x="43.18" y="31.75"/>
 <vertex x="43.18" y="40.64"/>
 <vertex x="39.37" y="44.45"/>
@@
 <via x="1.27" y="21.59" extent="1-16" drill="1.5" diameter="2.54"/>
 <via x="119.38" y="21.59" extent="1-16" drill="1.5" diameter="2.54"/>
-<polygon width="0.4064" layer="1" spacing="0.4064" isolate="1.6764">
-<vertex x="10.16" y="25.4"/>
-<vertex x="-1.27" y="25.4"/>
-<vertex x="-3.81" y="22.86"/>
-<vertex x="-3.81" y="20.32"/>
-<vertex x="-1.27" y="17.78"/>
-<vertex x="10.16" y="17.78"/>
-<vertex x="12.7" y="20.32"/>
-<vertex x="12.7" y="22.86"/>
-</polygon>
-<via x="11.43" y="21.59" extent="1-16" drill="1.5" diameter="2.54"/>
-<polygon width="0.4064" layer="16" spacing="0.4064" isolate="1.9304" thermals="no">
-<vertex x="-2.54" y="44.45"/>
-<vertex x="-6.35" y="40.64"/>
-<vertex x="-6.35" y="2.54"/>
-<vertex x="-2.54" y="-1.27"/>
-<vertex x="118.11" y="-1.27"/>
-<vertex x="127" y="6.35"/>
-<vertex x="127" y="40.64"/>
-<vertex x="123.19" y="44.45"/>
-</polygon>
-<via x="101.6" y="21.59" extent="1-16" drill="1.5" diameter="2.54"/>
-<polygon width="0.4064" layer="1" spacing="0.4064" isolate="1.6764" thermals="no">
-<vertex x="120.65" y="24.13"/>
-<vertex x="121.92" y="22.86"/>
-<vertex x="121.92" y="20.32"/>
-<vertex x="120.65" y="19.05"/>
-<vertex x="111.76" y="19.05"/>
-<vertex x="109.22" y="16.51"/>
+<polygon width="0.4064" layer="1" thermals="no">
+<vertex x="99.06" y="24.13"/>
+<vertex x="-3.81" y="24.13"/>
+<vertex x="-5.08" y="22.86"/>
+<vertex x="-5.08" y="20.32"/>
+<vertex x="-3.81" y="19.05"/>
+<vertex x="99.06" y="19.05"/>
 <vertex x="101.6" y="16.51"/>
-<vertex x="99.06" y="19.05"/>
-<vertex x="99.06" y="24.13"/>
+<vertex x="107.95" y="16.51"/>
+<vertex x="110.49" y="19.05"/>
+<vertex x="124.46" y="19.05"/>
+<vertex x="125.73" y="20.32"/>
+<vertex x="125.73" y="22.86"/>
+<vertex x="124.46" y="24.13"/>
+<vertex x="110.49" y="24.13"/>
+<vertex x="107.95" y="26.67"/>
 <vertex x="101.6" y="26.67"/>
-<vertex x="109.22" y="26.67"/>
-<vertex x="111.76" y="24.13"/>
-</polygon>
-</signal>
+</polygon>
+</signal>
