File: EAGLE/projects/PS/PS.sch (EAGLE design)
At the start: 5 parts

Commit message: input
Connections:
- removed net N$4: X2-2.KL, X3-1.KL
- new net VTHRU: L1.2, X3-1.KL
- net VIN: now also X3-2.KL; no longer L1.2
- net VOUT: now also X2-2.KL; no longer X3-2.KL
Other:
- moved on the sheet: L1, R1, X3-1, X3-2
Changed lines of the file:
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@@
 <setting verticaltext="up"/>
 </settings>
-<grid distance="0.1" unitdist="inch" unit="inch" style="lines" multiple="1" display="yes" altdistance="0.01" altunitdist="inch" altunit="inch"/>
+<grid distance="0.1" unitdist="inch" unit="inch" style="lines" multiple="1" display="no" altdistance="0.01" altunitdist="inch" altunit="inch"/>
 <layers>
 <layer number="1" name="Top" color="4" fill="1" visible="no" active="no"/>
@@
 <instance part="X2" gate="-1" x="40.64" y="53.34" rot="R180"/>
 <instance part="X2" gate="-2" x="40.64" y="68.58" rot="R180"/>
-<instance part="L1" gate="G$1" x="-5.08" y="68.58" rot="R180"/>
-<instance part="X3" gate="-1" x="27.94" y="68.58"/>
-<instance part="X3" gate="-2" x="12.7" y="68.58" rot="R180"/>
-<instance part="R1" gate="G$1" x="5.08" y="60.96" rot="R90"/>
+<instance part="L1" gate="G$1" x="22.86" y="68.58" rot="R180"/>
+<instance part="X3" gate="-1" x="7.62" y="68.58"/>
+<instance part="X3" gate="-2" x="-7.62" y="68.58" rot="R180"/>
+<instance part="R1" gate="G$1" x="33.02" y="60.96" rot="R90"/>
 </instances>
 <busses>
 </busses>
 <nets>
-<net name="VIN" class="0">
-<segment>
-<pinref part="X1" gate="-1" pin="KL"/>
-<pinref part="L1" gate="G$1" pin="2"/>
-<wire x1="-15.24" y1="68.58" x2="-12.7" y2="68.58" width="0.1524" layer="91"/>
-</segment>
-</net>
 <net name="GND" class="0">
 <segment>
 <pinref part="X1" gate="-2" pin="KL"/>
 <pinref part="X2" gate="-1" pin="KL"/>
-<wire x1="-15.24" y1="53.34" x2="5.08" y2="53.34" width="0.1524" layer="91"/>
+<wire x1="-15.24" y1="53.34" x2="33.02" y2="53.34" width="0.1524" layer="91"/>
 <pinref part="R1" gate="G$1" pin="1"/>
-<wire x1="5.08" y1="53.34" x2="35.56" y2="53.34" width="0.1524" layer="91"/>
-<wire x1="5.08" y1="55.88" x2="5.08" y2="53.34" width="0.1524" layer="91"/>
-<junction x="5.08" y="53.34"/>
+<wire x1="33.02" y1="53.34" x2="35.56" y2="53.34" width="0.1524" layer="91"/>
+<wire x1="33.02" y1="55.88" x2="33.02" y2="53.34" width="0.1524" layer="91"/>
+<junction x="33.02" y="53.34"/>
 </segment>
 </net>
@@
 <segment>
 <pinref part="L1" gate="G$1" pin="1"/>
-<pinref part="X3" gate="-2" pin="KL"/>
-<wire x1="2.54" y1="68.58" x2="5.08" y2="68.58" width="0.1524" layer="91"/>
+<wire x1="30.48" y1="68.58" x2="33.02" y2="68.58" width="0.1524" layer="91"/>
 <pinref part="R1" gate="G$1" pin="2"/>
-<wire x1="5.08" y1="68.58" x2="7.62" y2="68.58" width="0.1524" layer="91"/>
-<wire x1="5.08" y1="66.04" x2="5.08" y2="68.58" width="0.1524" layer="91"/>
-<junction x="5.08" y="68.58"/>
+<wire x1="33.02" y1="66.04" x2="33.02" y2="68.58" width="0.1524" layer="91"/>
+<pinref part="X2" gate="-2" pin="KL"/>
+<wire x1="33.02" y1="68.58" x2="35.56" y2="68.58" width="0.1524" layer="91"/>
+<junction x="33.02" y="68.58"/>
 </segment>
 </net>
-<net name="N$4" class="0">
+<net name="VIN" class="0">
+<segment>
+<pinref part="X1" gate="-1" pin="KL"/>
+<pinref part="X3" gate="-2" pin="KL"/>
+<wire x1="-15.24" y1="68.58" x2="-12.7" y2="68.58" width="0.1524" layer="91"/>
+</segment>
+</net>
+<net name="VTHRU" class="0">
 <segment>
 <pinref part="X3" gate="-1" pin="KL"/>
-<pinref part="X2" gate="-2" pin="KL"/>
-<wire x1="33.02" y1="68.58" x2="35.56" y2="68.58" width="0.1524" layer="91"/>
+<pinref part="L1" gate="G$1" pin="2"/>
+<wire x1="12.7" y1="68.58" x2="15.24" y2="68.58" width="0.1524" layer="91"/>
 </segment>
 </net>

Commit message: changes
Parts:
- added J1, J2: J10MM, jumper:J10MM
Connections:
- net VTHRU renamed VCAPS
- new net N$3: J1.2, J2.1, X3-2.KL
- net VIN: now also J1.1, J2.2; no longer X3-2.KL
Other:
- moved on the sheet: X1-1, X1-2
Changed lines of the file:
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@@
 <setting verticaltext="up"/>
 </settings>
-<grid distance="0.1" unitdist="inch" unit="inch" style="lines" multiple="1" display="no" altdistance="0.01" altunitdist="inch" altunit="inch"/>
+<grid distance="0.1" unitdist="inch" unit="inch" style="lines" multiple="1" display="yes" altdistance="0.01" altunitdist="inch" altunit="inch"/>
 <layers>
 <layer number="1" name="Top" color="4" fill="1" visible="no" active="no"/>
@@
 <part name="X3" library="con-wago-508" deviceset="W237-02P" device=""/>
 <part name="R1" library="resistor-power" deviceset="R" device="AC04"/>
+<part name="J1" library="jumper" deviceset="J" device="10MM"/>
+<part name="J2" library="jumper" deviceset="J" device="10MM"/>
 </parts>
 <sheets>
@@
 </plain>
 <instances>
-<instance part="X1" gate="-1" x="-20.32" y="68.58"/>
-<instance part="X1" gate="-2" x="-20.32" y="53.34"/>
+<instance part="X1" gate="-1" x="-38.1" y="68.58"/>
+<instance part="X1" gate="-2" x="-38.1" y="53.34"/>
 <instance part="X2" gate="-1" x="40.64" y="53.34" rot="R180"/>
 <instance part="X2" gate="-2" x="40.64" y="68.58" rot="R180"/>
@@
 <instance part="X3" gate="-2" x="-7.62" y="68.58" rot="R180"/>
 <instance part="R1" gate="G$1" x="33.02" y="60.96" rot="R90"/>
+<instance part="J1" gate="1" x="-22.86" y="68.58"/>
+<instance part="J2" gate="1" x="-22.86" y="60.96" rot="R180"/>
 </instances>
 <busses>
@@
 <net name="GND" class="0">
 <segment>
-<pinref part="X1" gate="-2" pin="KL"/>
 <pinref part="X2" gate="-1" pin="KL"/>
-<wire x1="-15.24" y1="53.34" x2="33.02" y2="53.34" width="0.1524" layer="91"/>
 <pinref part="R1" gate="G$1" pin="1"/>
 <wire x1="33.02" y1="53.34" x2="35.56" y2="53.34" width="0.1524" layer="91"/>
 <wire x1="33.02" y1="55.88" x2="33.02" y2="53.34" width="0.1524" layer="91"/>
+<pinref part="X1" gate="-2" pin="KL"/>
+<wire x1="-33.02" y1="53.34" x2="33.02" y2="53.34" width="0.1524" layer="91"/>
 <junction x="33.02" y="53.34"/>
 </segment>
@@
 </segment>
 </net>
-<net name="VIN" class="0">
-<segment>
-<pinref part="X1" gate="-1" pin="KL"/>
-<pinref part="X3" gate="-2" pin="KL"/>
-<wire x1="-15.24" y1="68.58" x2="-12.7" y2="68.58" width="0.1524" layer="91"/>
-</segment>
-</net>
-<net name="VTHRU" class="0">
+<net name="VCAPS" class="0">
 <segment>
 <pinref part="X3" gate="-1" pin="KL"/>
@@
 </segment>
 </net>
+<net name="N$3" class="0">
+<segment>
+<pinref part="J1" gate="1" pin="2"/>
+<pinref part="X3" gate="-2" pin="KL"/>
+<wire x1="-17.78" y1="68.58" x2="-15.24" y2="68.58" width="0.1524" layer="91"/>
+<wire x1="-15.24" y1="68.58" x2="-12.7" y2="68.58" width="0.1524" layer="91"/>
+<wire x1="-15.24" y1="68.58" x2="-15.24" y2="60.96" width="0.1524" layer="91"/>
+<junction x="-15.24" y="68.58"/>
+<pinref part="J2" gate="1" pin="1"/>
+<wire x1="-15.24" y1="60.96" x2="-17.78" y2="60.96" width="0.1524" layer="91"/>
+</segment>
+</net>
+<net name="VIN" class="0">
+<segment>
+<pinref part="J2" gate="1" pin="2"/>
+<wire x1="-27.94" y1="60.96" x2="-30.48" y2="60.96" width="0.1524" layer="91"/>
+<wire x1="-30.48" y1="60.96" x2="-30.48" y2="68.58" width="0.1524" layer="91"/>
+<pinref part="J1" gate="1" pin="1"/>
+<wire x1="-30.48" y1="68.58" x2="-27.94" y2="68.58" width="0.1524" layer="91"/>
+<pinref part="X1" gate="-1" pin="KL"/>
+<wire x1="-30.48" y1="68.58" x2="-33.02" y2="68.58" width="0.1524" layer="91"/>
+<junction x="-30.48" y="68.58"/>
+</segment>
+</net>

Commit message: a lot
Parts:
- added X4: (no value), con-wago-508:W237-02P
Connections:
- net N$3: now also X4-1.KL
- net VIN: now also X4-2.KL
Changed lines of the file:
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@@
 <setting verticaltext="up"/>
 </settings>
-<grid distance="0.1" unitdist="inch" unit="inch" style="lines" multiple="1" display="yes" altdistance="0.01" altunitdist="inch" altunit="inch"/>
+<grid distance="0.1" unitdist="inch" unit="inch" style="lines" multiple="1" display="no" altdistance="0.01" altunitdist="inch" altunit="inch"/>
 <layers>
 <layer number="1" name="Top" color="4" fill="1" visible="no" active="no"/>
@@
 <part name="J1" library="jumper" deviceset="J" device="10MM"/>
 <part name="J2" library="jumper" deviceset="J" device="10MM"/>
+<part name="X4" library="con-wago-508" deviceset="W237-02P" device=""/>
 </parts>
 <sheets>
@@
 <instance part="J1" gate="1" x="-22.86" y="68.58"/>
 <instance part="J2" gate="1" x="-22.86" y="60.96" rot="R180"/>
+<instance part="X4" gate="-1" x="-20.32" y="83.82" rot="R270"/>
+<instance part="X4" gate="-2" x="-25.4" y="83.82" rot="R270"/>
 </instances>
 <busses>
@@
 <pinref part="J2" gate="1" pin="1"/>
 <wire x1="-15.24" y1="60.96" x2="-17.78" y2="60.96" width="0.1524" layer="91"/>
+<wire x1="-15.24" y1="68.58" x2="-15.24" y2="76.2" width="0.1524" layer="91"/>
+<pinref part="X4" gate="-1" pin="KL"/>
+<wire x1="-15.24" y1="76.2" x2="-20.32" y2="76.2" width="0.1524" layer="91"/>
+<wire x1="-20.32" y1="76.2" x2="-20.32" y2="78.74" width="0.1524" layer="91"/>
 </segment>
 </net>
@@
 <wire x1="-30.48" y1="68.58" x2="-33.02" y2="68.58" width="0.1524" layer="91"/>
 <junction x="-30.48" y="68.58"/>
+<wire x1="-30.48" y1="68.58" x2="-30.48" y2="76.2" width="0.1524" layer="91"/>
+<pinref part="X4" gate="-2" pin="KL"/>
+<wire x1="-30.48" y1="76.2" x2="-25.4" y2="76.2" width="0.1524" layer="91"/>
+<wire x1="-25.4" y1="76.2" x2="-25.4" y2="78.74" width="0.1524" layer="91"/>
 </segment>
 </net>
