File: EAGLE/projects/gain_mute/gain_mute.brd (EAGLE design)
At the start: 50 x 50 mm, 31 parts, among them Q1 2N3820, U1 NE5532P

Commit message: stuff
Parts:
- removed JP1, JP2, JP3, JP4, JP5: (no value), pinhead:1X02
- removed R6: 100k, rcl:R1206
- added +15, -15, AUX, IN, MUTE, OUT: (no value), pinhead:1X02
- added C7, C8: (no value), rcl:C050-024X044
- added DELAY: 10k, pot:3223J
- added R14: 25k, rcl:0207/7
- added R15: 50k, rcl:0207/7
- C1, C2: value (none) -> 0.1u
- C3, C4: value (none) -> 22-33u
- C6: value (none) -> 10u
- D1: value 3.6V Zener -> 3.6V
- D2: value 3.6V Zener -> 1n4002
- R10, R12: value 20k -> 25k
- R11: value 10k -> 12k
- R13: value 30k -> 35k
- moved R13 129.6 mm to (43.2, 19.1), turned to 270 degrees
- moved R12 123.7 mm to (40.0, 19.1), flipped to the bottom, turned to 270 degrees
- moved JP6 123.6 mm to (39.4, 10.8)
- moved R8 118.7 mm to (43.2, 29.2), turned to 180 degrees
- moved R11 117.8 mm to (36.8, 19.1), turned to 270 degrees
- moved C7_BP1 115.0 mm to (39.4, 36.8), turned to 180 degrees
- moved R10 112.9 mm to (33.7, 26.7)
- moved R3 80.4 mm to (24.1, 38.1)
- moved C7_BP 79.6 mm to (29.8, 43.2), turned to 45 degrees
- moved R4 79.4 mm to (22.2, 33.0)
- moved C6 75.6 mm to (12.7, 26.7), turned to 270 degrees
- moved D2 74.6 mm to (11.4, 34.3), turned to 180 degrees
- moved C2 73.5 mm to (30.5, 22.2), flipped to the bottom
- moved Q1 71.2 mm to (30.5, 33.0)
- moved C1 60.0 mm to (21.6, 22.2), flipped to the bottom
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Connections:
- removed net N$16: U1.6, U1.7
- new net N$17: AUX.1, C8.2, R15.2, U1.7
- new net N$18: C8.1, R14.2, R15.1, U1.6
- net AGND: now also AUX.2, IN.1, OUT.2; no longer JP1.1, JP2.2
- net GND: now also +15.2, -15.2, MUTE.1; no longer JP3.2, JP4.2, JP5.1
- net N$1: now also +15.1; no longer JP3.1
- net N$10: now also R14.1
- net N$11: now also C7.1, R11.1, R12.1, R13.1; no longer JP6.2, JP6.4, JP6.6
- net N$12: now also JP6.4, R12.2; no longer JP6.5, R13.1
- net N$13: now also JP6.6, R13.2; no longer JP6.3, R12.1
- net N$14: now also JP6.2, R11.2; no longer JP6.1, R11.1
- net N$15: now also C7.2, JP6.1, JP6.3, JP6.5, OUT.1; no longer JP2.1, R11.2, R12.2, R13.2
- net N$2: now also IN.2; no longer JP1.2
- net N$3: now also DELAY.3, MUTE.2; no longer JP5.2, R6.2
- net N$4: now also -15.1; no longer JP4.1
- net N$6: now also DELAY.1, DELAY.2; no longer R6.1
Routing:
- net AGND: track 0.00 -> 74.4 mm
- net +15V: track 0.00 -> 54.1 mm
- net GND: track 0.00 -> 52.4 mm, vias 0 -> 1
- net -15V: track 0.00 -> 40.4 mm
- net N$5: track 0.00 -> 32.7 mm
- net N$17: track 0.00 -> 26.7 mm
- net N$10: track 0.00 -> 26.5 mm
- net N$11: track 0.00 -> 25.4 mm
- net N$18: track 0.00 -> 20.8 mm
- net N$15: track 0.00 -> 19.5 mm
- net N$6: track 0.00 -> 18.4 mm
- net +5V/2: track 0.00 -> 17.5 mm
- net N$7: track 0.00 -> 13.9 mm
- net N$3: track 0.00 -> 8.32 mm
- net N$9: track 0.00 -> 7.93 mm
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- added copper zone on layer 16, net GND
Other:
- board size 50 x 50 mm -> 49.5 x 49.5 mm
