File: EAGLE/projects/gain_mute/gain_mute.sch (EAGLE design)
At the start: 31 parts, among them Q1 2N3820, U1 NE5532P

Commit message: stuff
Parts:
- removed JP5: (no value), pinhead:PINHD-1X2
- removed R6: 100k, rcl:R-US_R1206
- added AUX, MUTE: (no value), pinhead:PINHD-1X2
- added C7, C8: (no value), rcl:C-US050-024X044
- added DELAY: 10k, pot:TRIM_US-3223J
- added R14: 25k, rcl:R-US_0207/7
- added R15: 50k, rcl:R-US_0207/7
- C1, C2: value (none) -> 0.1u
- C3, C4: value (none) -> 22-33u
- C6: value (none) -> 10u
- D1: value 3.6V Zener -> 3.6V
- D2: value 3.6V Zener -> 1n4002
- R10, R12: value 20k -> 25k
- R11: value 10k -> 12k
- R13: value 30k -> 35k
- renumbered JP1 to IN, JP2 to OUT, JP3 to +15, JP4 to -15
Connections:
- removed net N$16: U1.2IN-, U1.2OUT
- new net N$17: AUX.1, C8.2, R15.2, U1.2OUT
- new net N$18: C8.1, R14.2, R15.1, U1.2IN-
- net AGND: now also AUX.2
- net GND: now also MUTE.1; no longer JP5.1
- net N$10: now also R14.1
- net N$11: now also C7.1, R11.1, R12.1, R13.1; no longer JP6.2, JP6.4, JP6.6
- net N$12: now also JP6.4, R12.2; no longer JP6.5, R13.1
- net N$13: now also JP6.6, R13.2; no longer JP6.3, R12.1
- net N$14: now also JP6.2, R11.2; no longer JP6.1, R11.1
- net N$15: now also C7.2, JP6.1, JP6.3, JP6.5; no longer R11.2, R12.2, R13.2
- net N$3: now also DELAY.E, MUTE.2; no longer JP5.2, R6.2
- net N$6: now also DELAY.A, DELAY.S; no longer R6.1
Other:
- moved on the sheet: JP6, R11, R12, R13, R8
