File: EAGLE/projects/lm317 reg/board.brd (EAGLE design)
At the start: 49.5 x 49.5 mm, 15 parts

Commit message: a lot
Parts:
- added JP1: (no value), pinhead:1X02
- added R5: 4K, rcl:R1206
- added R6: 1K, rcl:R1206
- R4: value 3.9k -> 3.9K
- moved D2 7.62 mm to (24.8, 36.8)
- moved R4 7.62 mm to (24.8, 30.5)
- moved R3 2.84 mm to (19.1, 21.6)
- turned C4 to 225 degrees
Connections:
- new net N$5: JP1.1, R5.1, R6.2
- net GND: now also JP1.2, R6.1
- net N$6: now also R5.2
Routing:
- net N$5: track 0.00 -> 14.7 mm
- net GND: track 30.7 -> 42.6 mm
- net N$6: track 87.0 -> 89.4 mm
- net N$3: track 36.4 -> 34.4 mm
- net N$1: track 77.1 -> 75.1 mm

Commit message: stuff
Parts:
- moved C1 1.27 mm to (16.5, 39.4)
- moved C3 1.27 mm to (33.0, 39.4)
- moved C5 1.27 mm to (39.4, 25.4)
- moved D1 1.27 mm to (43.2, 10.2)
- moved VIN 1.27 mm to (7.62, 39.4)
- moved VOUT 1.27 mm to (41.9, 39.4)
- moved C2 1.27 mm to (16.5, 6.35)
- moved R1 1.27 mm to (8.89, 7.62)
- moved C4 1.27 mm to (8.89, 26.7)
- moved R2 1.27 mm to (8.89, 16.5)
Routing:
- net N$1: track 75.1 -> 71.7 mm
- net N$4: track 10.7 -> 8.89 mm
