File: EAGLE/projects/lm317 reg/board.sch (EAGLE design)
At the start: 1 part

Commit message: LM317 Reg
Parts:
- added C1: 0.1u, rcl:C-USC1206
- added C2: 10u, rcl:CPOL-USE2-5
- added C3: 1u, rcl:C-USC1206
- added C4: 220u, rcl:CPOL-USE5-10.5
- added C5: 470u, rcl:CPOL-USE5-13
- added D1: 1N4004, diode:1N4004
- added D2: (no value), SparkFun-LED:LED1206
- added R1: 5K, rcl:R-TRIMM3296W
- added R2: 500, rcl:R-TRIMM3296W
- added R3: 240, rcl:R-US_0309/10
- added R4: 3.9k, rcl:R-US_R1206
- added REG: (no value), con-wago-508:W237-3E
- added VIN, VOUT: (no value), con-wago-508:W237-02P
- IC1: device v-reg:LM317-TO3 -> v-reg:LM317TS
Connections:
- new net GND: C1.2, C2.-, C3.2, C4.-, C5.-, D2.C, R2.E, VIN-1.KL, VOUT-2.KL
- new net N$1: C1.1, C4.+, D1.C, IC1.IN, REG-3.KL, VIN-2.KL
- new net N$2: D2.A, R4.1
- new net N$3: C2.+, IC1.ADJ, R1.A, R1.S, R3.1, REG-1.KL
- new net N$4: R1.E, R2.A, R2.S
- new net N$6: C3.1, C5.+, D1.A, IC1.OUT, R3.2, R4.2, REG-2.KL, VOUT-1.KL

Commit message: a lot
Parts:
- added JP1: (no value), pinhead:PINHD-1X2
- added R5: 4K, rcl:R-US_R1206
- added R6: 1K, rcl:R-US_R1206
- R4: value 3.9k -> 3.9K
Connections:
- new net N$5: JP1.1, R5.1, R6.2
- net GND: now also JP1.2, R6.1
- net N$6: now also R5.2
Other:
- moved on the sheet: VOUT-1, VOUT-2
Changed lines of the file:
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@@
 <setting verticaltext="up"/>
 </settings>
-<grid distance="0.1" unitdist="inch" unit="inch" style="lines" multiple="1" display="no" altdistance="0.01" altunitdist="inch" altunit="inch"/>
+<grid distance="0.1" unitdist="inch" unit="inch" style="lines" multiple="1" display="yes" altdistance="0.01" altunitdist="inch" altunit="inch"/>
 <layers>
 <layer number="1" name="Top" color="4" fill="1" visible="no" active="no"/>
@@
 <part name="VIN" library="con-wago-508" deviceset="W237-02P" device=""/>
 <part name="VOUT" library="con-wago-508" deviceset="W237-02P" device=""/>
-<part name="R4" library="rcl" deviceset="R-US_" device="R1206" value="3.9k"/>
+<part name="R4" library="rcl" deviceset="R-US_" device="R1206" value="3.9K"/>
 <part name="D2" library="SparkFun-LED" deviceset="LED" device="1206"/>
 <part name="GND1" library="supply1" deviceset="GND" device=""/>
+<part name="R5" library="rcl" deviceset="R-US_" device="R1206" value="4K"/>
+<part name="R6" library="rcl" deviceset="R-US_" device="R1206" value="1K"/>
+<part name="JP1" library="pinhead" deviceset="PINHD-1X2" device=""/>
 </parts>
 <sheets>
@@
 <instance part="VIN" gate="-1" x="0" y="58.42"/>
 <instance part="VIN" gate="-2" x="0" y="63.5"/>
-<instance part="VOUT" gate="-1" x="99.06" y="63.5" rot="R180"/>
-<instance part="VOUT" gate="-2" x="99.06" y="58.42" rot="R180"/>
+<instance part="VOUT" gate="-1" x="109.22" y="63.5" rot="R180"/>
+<instance part="VOUT" gate="-2" x="109.22" y="58.42" rot="R180"/>
 <instance part="R4" gate="G$1" x="83.82" y="55.88" rot="R90"/>
 <instance part="D2" gate="G$1" x="83.82" y="45.72"/>
-<instance part="GND1" gate="1" x="66.04" y="30.48"/>
+<instance part="GND1" gate="1" x="66.04" y="27.94"/>
+<instance part="R5" gate="G$1" x="93.98" y="55.88" rot="R90"/>
+<instance part="R6" gate="G$1" x="93.98" y="40.64" rot="R90"/>
+<instance part="JP1" gate="G$1" x="116.84" y="45.72"/>
 </instances>
 <busses>
@@
 <pinref part="C2" gate="G$1" pin="-"/>
 <wire x1="43.18" y1="17.78" x2="55.88" y2="17.78" width="0.1524" layer="91"/>
-<wire x1="55.88" y1="17.78" x2="55.88" y2="35.56" width="0.1524" layer="91"/>
+<wire x1="55.88" y1="17.78" x2="55.88" y2="33.02" width="0.1524" layer="91"/>
 <pinref part="C3" gate="G$1" pin="2"/>
-<wire x1="55.88" y1="35.56" x2="55.88" y2="38.1" width="0.1524" layer="91"/>
+<wire x1="55.88" y1="33.02" x2="55.88" y2="38.1" width="0.1524" layer="91"/>
 <wire x1="66.04" y1="53.34" x2="66.04" y2="50.8" width="0.1524" layer="91"/>
 <pinref part="C5" gate="G$1" pin="-"/>
@@
 <wire x1="73.66" y1="50.8" x2="66.04" y2="50.8" width="0.1524" layer="91"/>
 <junction x="66.04" y="50.8"/>
-<wire x1="55.88" y1="35.56" x2="66.04" y2="35.56" width="0.1524" layer="91"/>
-<wire x1="66.04" y1="35.56" x2="66.04" y2="50.8" width="0.1524" layer="91"/>
-<junction x="55.88" y="35.56"/>
+<wire x1="55.88" y1="33.02" x2="66.04" y2="33.02" width="0.1524" layer="91"/>
+<wire x1="66.04" y1="33.02" x2="66.04" y2="50.8" width="0.1524" layer="91"/>
+<junction x="55.88" y="33.02"/>
 <pinref part="D2" gate="G$1" pin="C"/>
-<wire x1="66.04" y1="35.56" x2="83.82" y2="35.56" width="0.1524" layer="91"/>
-<wire x1="83.82" y1="35.56" x2="83.82" y2="38.1" width="0.1524" layer="91"/>
-<junction x="66.04" y="35.56"/>
-<wire x1="83.82" y1="38.1" x2="83.82" y2="40.64" width="0.1524" layer="91"/>
+<wire x1="66.04" y1="33.02" x2="83.82" y2="33.02" width="0.1524" layer="91"/>
+<junction x="66.04" y="33.02"/>
+<wire x1="83.82" y1="33.02" x2="83.82" y2="40.64" width="0.1524" layer="91"/>
 <pinref part="VOUT" gate="-2" pin="KL"/>
-<wire x1="93.98" y1="58.42" x2="91.44" y2="58.42" width="0.1524" layer="91"/>
-<wire x1="83.82" y1="38.1" x2="91.44" y2="38.1" width="0.1524" layer="91"/>
-<wire x1="91.44" y1="38.1" x2="91.44" y2="58.42" width="0.1524" layer="91"/>
-<junction x="83.82" y="38.1"/>
+<wire x1="104.14" y1="58.42" x2="101.6" y2="58.42" width="0.1524" layer="91"/>
+<wire x1="83.82" y1="33.02" x2="93.98" y2="33.02" width="0.1524" layer="91"/>
+<wire x1="93.98" y1="33.02" x2="101.6" y2="33.02" width="0.1524" layer="91"/>
+<wire x1="101.6" y1="33.02" x2="101.6" y2="45.72" width="0.1524" layer="91"/>
+<junction x="83.82" y="33.02"/>
 <pinref part="GND1" gate="1" pin="GND"/>
-<wire x1="66.04" y1="33.02" x2="66.04" y2="35.56" width="0.1524" layer="91"/>
+<wire x1="101.6" y1="45.72" x2="101.6" y2="58.42" width="0.1524" layer="91"/>
+<wire x1="66.04" y1="30.48" x2="66.04" y2="33.02" width="0.1524" layer="91"/>
+<pinref part="R6" gate="G$1" pin="1"/>
+<wire x1="93.98" y1="35.56" x2="93.98" y2="33.02" width="0.1524" layer="91"/>
+<junction x="93.98" y="33.02"/>
+<pinref part="JP1" gate="G$1" pin="2"/>
+<wire x1="114.3" y1="45.72" x2="101.6" y2="45.72" width="0.1524" layer="91"/>
+<junction x="101.6" y="45.72"/>
 </segment>
 </net>
@@
 <wire x1="83.82" y1="63.5" x2="93.98" y2="63.5" width="0.1524" layer="91"/>
 <junction x="83.82" y="63.5"/>
+<wire x1="93.98" y1="63.5" x2="104.14" y2="63.5" width="0.1524" layer="91"/>
 <wire x1="53.34" y1="73.66" x2="53.34" y2="71.12" width="0.1524" layer="91"/>
 <junction x="53.34" y="63.5"/>
@@
 <wire x1="50.8" y1="71.12" x2="53.34" y2="71.12" width="0.1524" layer="91"/>
 <junction x="53.34" y="71.12"/>
-</segment>
-</net>
+<pinref part="R5" gate="G$1" pin="2"/>
+<wire x1="93.98" y1="60.96" x2="93.98" y2="63.5" width="0.1524" layer="91"/>
+<junction x="93.98" y="63.5"/>
+</segment>
+</net>
+<net name="N$5" class="0">
+<segment>
+<pinref part="R5" gate="G$1" pin="1"/>
+<pinref part="R6" gate="G$1" pin="2"/>
+<wire x1="93.98" y1="50.8" x2="93.98" y2="48.26" width="0.1524" layer="91"/>
+<pinref part="JP1" gate="G$1" pin="1"/>
+<wire x1="93.98" y1="48.26" x2="93.98" y2="45.72" width="0.1524" layer="91"/>
+<wire x1="114.3" y1="48.26" x2="93.98" y2="48.26" width="0.1524" layer="91"/>
+<junction x="93.98" y="48.26"/>
+</segment>
+</net>

Commit message: stuff
Changed lines of the file:
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@@
 <setting verticaltext="up"/>
 </settings>
-<grid distance="0.1" unitdist="inch" unit="inch" style="lines" multiple="1" display="yes" altdistance="0.01" altunitdist="inch" altunit="inch"/>
+<grid distance="0.1" unitdist="inch" unit="inch" style="lines" multiple="1" display="no" altdistance="0.01" altunitdist="inch" altunit="inch"/>
 <layers>
 <layer number="1" name="Top" color="4" fill="1" visible="no" active="no"/>
@@
 <net name="GND" class="0">
 <segment>
-<wire x1="43.18" y1="22.86" x2="43.18" y2="25.4" width="0.1524" layer="91"/>
-</segment>
-<segment>
 <pinref part="R2" gate="G$1" pin="E"/>
